File: Electronics/GNBoard_0.1/GNBoard/GNBoard.sch (KiCad schematic (older format))
At the start: 47 parts, among them K1 IR1, K10 IR4, K11 CNY_1, K12 CNY_2, K13 CNY_3, K14 CNY_4, K15 CNY_5, K16 CNY_6, K2 IR2, K3 SERVO_1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

Commit message: Updated value of the resistors for the battery voltage monitor
Parts:
- R1: value 62k -> 22k
- R5: value 20k -> 6k8
Changed lines of the file:
@@
 Sheet 1 1
 Title ""
-Date "14 jan 2014"
+Date "10 feb 2014"
 Rev ""
 Comp ""
@@
 P 1050 4000
 F 0 "R1" V 1130 4000 40  0000 C CNN
-F 1 "62k" V 1057 4001 40  0000 C CNN
+F 1 "22k" V 1057 4001 40  0000 C CNN
 F 2 "~" V 980 4000 30  0000 C CNN
 F 3 "~" H 1050 4000 30  0000 C CNN
@@
 P 1750 4000
 F 0 "R5" V 1830 4000 40  0000 C CNN
-F 1 "20k" V 1757 4001 40  0000 C CNN
+F 1 "6k8" V 1757 4001 40  0000 C CNN
 F 2 "~" V 1680 4000 30  0000 C CNN
 F 3 "~" H 1750 4000 30  0000 C CNN
