File: Electronics/GNBoard_1.0/GNBoard.kicad_pcb (KiCad board)
At the start: 2 copper layers, 80.8 x 55.4 mm, 58 parts, among them K1 IR1, K10 IR4, K11 CNY_1, K12 CNY_2, K13 CNY_3, K14 CNY_4, K2 IR2, K3 SERVO_1, K4 SERVO_2, K5 SERVO_3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

Commit message: Resized silkscreen texts, resistor values are now shown
Parts:
- R1, R12, R13, R14, R15, R16, R17, R18, R2, R3, R4, R5, R6, R7, R8, R9: footprint R3-LARGE_PADS -> R3-LARGE_PADS_CUSTOM
- R10, R11: value R -> 4k7; footprint R3-LARGE_PADS -> R3-LARGE_PADS_CUSTOM
Other:
- board text added: "+5v"
- board text added: "11"
- board text added: "12"
- board text added: "13"
- board text added: "20v"
- board text added: "3v3"
- board text added: "Analog:"
- board text added: "GNBoard for the GNBot (http://github.com/carlosgs/GNBot) by Carlos Garcia Saura (http://carlosgs.es)"
- board text added: "License: Creative Commons Attribution-ShareAlike 4.0 International"
- board text added: "RCGB"
- board text removed: "A11"
- board text removed: "A12"
- board text removed: "A13"
- board text removed: "A14"
- board text removed: "A15"
- board text removed: "http://carlosgs.es"

Commit message: Updated value of the resistors for the battery voltage monitor
Parts:
- R1: value 62k -> 22k
- R5: value 20k -> 6k8
Changed lines of the file:
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@@
       (effects (font (size 0.8382 0.8382) (thickness 0.1778)))
     )
-    (fp_text value 62k (at -1.4478 -0.0127) (layer F.SilkS)
+    (fp_text value 22k (at -1.4478 -0.0127) (layer F.SilkS)
       (effects (font (size 0.8382 0.8382) (thickness 0.1778)))
     )
@@
       (effects (font (size 0.8382 0.8382) (thickness 0.1778)))
     )
-    (fp_text value 20k (at -1.4478 -0.0127 270) (layer F.SilkS)
+    (fp_text value 6k8 (at -1.4478 -0.0127 270) (layer F.SilkS)
       (effects (font (size 0.8382 0.8382) (thickness 0.1778)))
     )
